Commit message: Update launch files, map configs, costmap params, and URDF model
- Adjust base_serial, my_lidar, static_tf, and test_amcl launch files
- Update navigation map (nav.pgm, nav.yaml)
- Tweak costmap common parameters
- Update mini_akm_robot URDF description

Co-Authored-By: Claude Opus 4.8 <noreply@anthropic.com>

File: src/ebot_description/urdf/mini_akm_robot.urdf (robot description, URDF)
Before this commit: robot wheeltec_robot, 5 links, 4 joints
Links:
- link base_link: geometry visual box size=0.23 0.11 0.05; visual sphere radius=0.02
